File: masterzen_tutorial_pcb_design/masterzen_tutorial_pcb_design.kicad_pcb (KiCad board)
At the start: 2 copper layers, 196 parts, among them SW1 SW_Push, SW10 F7, SW11 F8, SW12 F9, SW13 F10, SW14 F11, SW15 F12, SW16 Pause/SrLk, SW17 Delete/Insert, SW2 RotaryEncoder_Switch, SW20 1, SW21 2, SW22 3, SW23 4, SW24 5, SW25 6, SW26 7, SW27 8, SW28 9, SW29 0, SW3 ESC, SW30 j-, SW31 =, SW32 Backspace, SW33 Home, SW34 Tab, SW35 Q, SW36 W, SW37 E, SW38 R, SW39 T, SW4 F1, SW40 Y, SW41 U, SW42 I, SW43 O, SW44 P, SW45 [, SW46 ], SW47 \, SW48 Page Up, SW49 Caps Lock, SW5 F2, SW50 A, SW51 S, SW52 D, SW53 F, SW54 G, SW55 H, SW56 J, SW57 K, SW58 L, SW59 ;, SW6 F3, SW60 ', SW61 Enter, SW62 Page Down, SW63 Shift, SW64 Z, SW65 X, SW66 C, SW67 V, SW68 B, SW69 N, SW7 F4, SW70 M, SW71 ,, SW72 ., SW73 /, SW74 r Shift, SW75 Up Arrow, SW76 End, SW77 Ctrl, SW78 Win, SW79 Alt, SW8 F5, SW80 Spacebar, SW81 r Alt, SW82 Fn, SW83 r Ctrl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

Commit message: starting placing components on a pcb
Parts:
- removed the D16 at (275.5, 133.2)
- removed the D64 at (252.3, 129.9)
- removed the D67 at (252.3, 139.9)
- removed the D71 at (252.3, 153.3)
- removed the D72 at (252.3, 156.7)
- removed D76, D77, D78, D79, D80, D81, D82, D83, D84, D85: D, Diode_SMD:D_SOD-123
- removed the SW17 at (47.3, 71.1)
- removed the SW47 at (77.5, 176.7)
- removed the SW66 at (107.6, 131.4)
- removed the SW67 at (107.6, 146.5)
- removed the SW69 at (107.6, 176.7)
- removed SW77: Ctrl, Button_Switch_Keyboard:SW_Cherry_MX_1.00u_PCB
- removed SW78: Win, Button_Switch_Keyboard:SW_Cherry_MX_1.00u_PCB
- removed SW79: Alt, Button_Switch_Keyboard:SW_Cherry_MX_1.00u_PCB
- removed SW80: Spacebar, Button_Switch_Keyboard:SW_Cherry_MX_1.00u_PCB
- removed SW81: r Alt, Button_Switch_Keyboard:SW_Cherry_MX_1.00u_PCB
- removed SW82: Fn, Button_Switch_Keyboard:SW_Cherry_MX_1.00u_PCB
- removed SW83: r Ctrl, Button_Switch_Keyboard:SW_Cherry_MX_1.00u_PCB
- removed SW84: left, Button_Switch_Keyboard:SW_Cherry_MX_1.00u_PCB
- removed SW85: down, Button_Switch_Keyboard:SW_Cherry_MX_1.00u_PCB
- removed SW86: right, Button_Switch_Keyboard:SW_Cherry_MX_1.00u_PCB
- added D2: Caps Lock LED, LED_SMD:LED_0805_2012Metric_Pad1.15x1.40mm_HandSolder, B.Cu at (170.1, 172.0)
- added D31: D, Diode_SMD:D_SOD-123, B.Cu at (319.9, 84.9)
- added D61: D, Diode_SMD:D_SOD-123, B.Cu at (319.9, 123.0)
- added D70: D, Diode_SMD:D_SOD-123, B.Cu at (281.8, 142.1)
- added R2: 5.1k, Resistor_SMD:R_0805_2012Metric_Pad1.20x1.40mm_HandSolder, B.Cu at (178.0, 173.0)
- added R3: 5.1k, Resistor_SMD:R_0805_2012Metric_Pad1.20x1.40mm_HandSolder, B.Cu at (178.0, 176.0)
- added R7: 5.1k, Resistor_SMD:R_0805_2012Metric_Pad1.20x1.40mm_HandSolder, B.Cu at (178.0, 178.9)
- added SW31: Delete Insert, MX_Only:MXOnly-1U-NoLED, F.Cu at (323.1, 81.0)
- added SW46: PrtSc NmLk, MX_Only:MXOnly-1U-NoLED, F.Cu at (323.1, 100.0)
- added SW61: Pause ScrLk, MX_Only:MXOnly-1U-NoLED, F.Cu at (323.1, 119.1)
- SW10: value F7 -> & 7; footprint Button_Switch_Keyboard:SW_Cherry_MX_1.00u_PCB -> MX_Only:MXOnly-1U-NoLED
- SW11: value F8 -> * 8; footprint Button_Switch_Keyboard:SW_Cherry_MX_1.00u_PCB -> MX_Only:MXOnly-1U-NoLED
- SW12: value F9 -> ( 9; footprint Button_Switch_Keyboard:SW_Cherry_MX_1.00u_PCB -> MX_Only:MXOnly-1U-NoLED
- SW13: value F10 -> ) 0; footprint Button_Switch_Keyboard:SW_Cherry_MX_1.00u_PCB -> MX_Only:MXOnly-1U-NoLED
- SW14: value F11 -> _ -; footprint Button_Switch_Keyboard:SW_Cherry_MX_1.00u_PCB -> MX_Only:MXOnly-1U-NoLED
- SW15: value F12 -> + =; footprint Button_Switch_Keyboard:SW_Cherry_MX_1.00u_PCB -> MX_Only:MXOnly-1U-NoLED
- SW16: value Pause/SrLk -> Backspace; footprint Button_Switch_Keyboard:SW_Cherry_MX_1.00u_PCB -> MX_Only:MXOnly-2U-NoLED
- SW17: renamed from SW19; value ~ -> Tab; footprint Button_Switch_Keyboard:SW_Cherry_MX_1.00u_PCB -> MX_Only:MXOnly-1.5U-NoLED
- SW18: renamed from SW20; value 1 -> Q; footprint Button_Switch_Keyboard:SW_Cherry_MX_1.00u_PCB -> MX_Only:MXOnly-1U-NoLED
- SW19: renamed from SW21; value 2 -> W; footprint Button_Switch_Keyboard:SW_Cherry_MX_1.00u_PCB -> MX_Only:MXOnly-1U-NoLED
- SW20: renamed from SW22; value 3 -> E; footprint Button_Switch_Keyboard:SW_Cherry_MX_1.00u_PCB -> MX_Only:MXOnly-1U-NoLED
- SW21: renamed from SW23; value 4 -> R; footprint Button_Switch_Keyboard:SW_Cherry_MX_1.00u_PCB -> MX_Only:MXOnly-1U-NoLED
- SW22: renamed from SW24; value 5 -> T; footprint Button_Switch_Keyboard:SW_Cherry_MX_1.00u_PCB -> MX_Only:MXOnly-1U-NoLED
- SW23: renamed from SW25; value 6 -> Y; footprint Button_Switch_Keyboard:SW_Cherry_MX_1.00u_PCB -> MX_Only:MXOnly-1U-NoLED
- SW24: renamed from SW26; value 7 -> U; footprint Button_Switch_Keyboard:SW_Cherry_MX_1.00u_PCB -> MX_Only:MXOnly-1U-NoLED
- SW25: renamed from SW27; value 8 -> I; footprint Button_Switch_Keyboard:SW_Cherry_MX_1.00u_PCB -> MX_Only:MXOnly-1U-NoLED
- SW26: renamed from SW28; value 9 -> O; footprint Button_Switch_Keyboard:SW_Cherry_MX_1.00u_PCB -> MX_Only:MXOnly-1U-NoLED
- SW27: renamed from SW29; value 0 -> P; footprint Button_Switch_Keyboard:SW_Cherry_MX_1.00u_PCB -> MX_Only:MXOnly-1U-NoLED
- SW28: renamed from SW30; value j- -> [; footprint Button_Switch_Keyboard:SW_Cherry_MX_1.00u_PCB -> MX_Only:MXOnly-1U-NoLED
- SW29: renamed from SW31; value = -> ]; footprint Button_Switch_Keyboard:SW_Cherry_MX_1.00u_PCB -> MX_Only:MXOnly-1U-NoLED
- SW3, SW62: footprint Button_Switch_Keyboard:SW_Cherry_MX_1.00u_PCB -> MX_Only:MXOnly-1U-NoLED
- SW30: renamed from SW32; value Backspace -> \; footprint Button_Switch_Keyboard:SW_Cherry_MX_1.00u_PCB -> MX_Only:MXOnly-1.5U-NoLED
- SW32: renamed from SW33; footprint Button_Switch_Keyboard:SW_Cherry_MX_1.00u_PCB -> MX_Only:MXOnly-1U-NoLED
- SW33: renamed from SW34; value Tab -> Caps Lock; footprint Button_Switch_Keyboard:SW_Cherry_MX_1.00u_PCB -> MX_Only:MXOnly-1.75U-NoLED
- SW34: renamed from SW35; value Q -> A; footprint Button_Switch_Keyboard:SW_Cherry_MX_1.00u_PCB -> MX_Only:MXOnly-1U-NoLED
- SW35: renamed from SW36; value W -> S; footprint Button_Switch_Keyboard:SW_Cherry_MX_1.00u_PCB -> MX_Only:MXOnly-1U-NoLED
- SW36: renamed from SW37; value E -> D; footprint Button_Switch_Keyboard:SW_Cherry_MX_1.00u_PCB -> MX_Only:MXOnly-1U-NoLED
- SW37: renamed from SW38; value R -> F; footprint Button_Switch_Keyboard:SW_Cherry_MX_1.00u_PCB -> MX_Only:MXOnly-1U-NoLED
- SW38: renamed from SW39; value T -> G; footprint Button_Switch_Keyboard:SW_Cherry_MX_1.00u_PCB -> MX_Only:MXOnly-1U-NoLED
- SW39: renamed from SW40; value Y -> H; footprint Button_Switch_Keyboard:SW_Cherry_MX_1.00u_PCB -> MX_Only:MXOnly-1U-NoLED
- SW4: value F1 -> ! 1; footprint Button_Switch_Keyboard:SW_Cherry_MX_1.00u_PCB -> MX_Only:MXOnly-1U-NoLED
- SW40: renamed from SW41; value U -> J; footprint Button_Switch_Keyboard:SW_Cherry_MX_1.00u_PCB -> MX_Only:MXOnly-1U-NoLED
- SW41: renamed from SW42; value I -> K; footprint Button_Switch_Keyboard:SW_Cherry_MX_1.00u_PCB -> MX_Only:MXOnly-1U-NoLED
- SW42: renamed from SW43; value O -> L; footprint Button_Switch_Keyboard:SW_Cherry_MX_1.00u_PCB -> MX_Only:MXOnly-1U-NoLED
- SW43: renamed from SW44; value P -> :; footprint Button_Switch_Keyboard:SW_Cherry_MX_1.00u_PCB -> MX_Only:MXOnly-1U-NoLED
- SW44: renamed from SW45; value [ -> :; footprint Button_Switch_Keyboard:SW_Cherry_MX_1.00u_PCB -> MX_Only:MXOnly-1U-NoLED
- SW45: renamed from SW46; value ] -> Enter; footprint Button_Switch_Keyboard:SW_Cherry_MX_1.00u_PCB -> MX_Only:MXOnly-2.25U-NoLED
- SW47: renamed from SW48; footprint Button_Switch_Keyboard:SW_Cherry_MX_1.00u_PCB -> MX_Only:MXOnly-1U-NoLED
- SW48: renamed from SW49; value Caps Lock -> left Shift; footprint Button_Switch_Keyboard:SW_Cherry_MX_1.00u_PCB -> MX_Only:MXOnly-2.25U-NoLED
- SW49: renamed from SW50; value A -> Z; footprint Button_Switch_Keyboard:SW_Cherry_MX_1.00u_PCB -> MX_Only:MXOnly-1U-NoLED
- SW5: value F2 -> @ 2; footprint Button_Switch_Keyboard:SW_Cherry_MX_1.00u_PCB -> MX_Only:MXOnly-1U-NoLED
- SW50: renamed from SW51; value S -> X; footprint Button_Switch_Keyboard:SW_Cherry_MX_1.00u_PCB -> MX_Only:MXOnly-1U-NoLED
- SW51: renamed from SW52; value D -> C; footprint Button_Switch_Keyboard:SW_Cherry_MX_1.00u_PCB -> MX_Only:MXOnly-1U-NoLED
- SW52: renamed from SW53; value F -> V; footprint Button_Switch_Keyboard:SW_Cherry_MX_1.00u_PCB -> MX_Only:MXOnly-1U-NoLED
- SW53: renamed from SW54; value G -> B; footprint Button_Switch_Keyboard:SW_Cherry_MX_1.00u_PCB -> MX_Only:MXOnly-1U-NoLED
- SW54: renamed from SW55; value H -> N; footprint Button_Switch_Keyboard:SW_Cherry_MX_1.00u_PCB -> MX_Only:MXOnly-1U-NoLED
- SW55: renamed from SW56; value J -> M; footprint Button_Switch_Keyboard:SW_Cherry_MX_1.00u_PCB -> MX_Only:MXOnly-1U-NoLED
- SW56: renamed from SW57; value K -> ,; footprint Button_Switch_Keyboard:SW_Cherry_MX_1.00u_PCB -> MX_Only:MXOnly-1U-NoLED
- SW57: renamed from SW58; value L -> .; footprint Button_Switch_Keyboard:SW_Cherry_MX_1.00u_PCB -> MX_Only:MXOnly-1U-NoLED
- SW58: renamed from SW59; value ; -> /; footprint Button_Switch_Keyboard:SW_Cherry_MX_1.00u_PCB -> MX_Only:MXOnly-1U-NoLED
- SW59: renamed from SW60; value ' -> right shift; footprint Button_Switch_Keyboard:SW_Cherry_MX_1.00u_PCB -> MX_Only:MXOnly-1.75U-NoLED
- SW6: value F3 -> # 3; footprint Button_Switch_Keyboard:SW_Cherry_MX_1.00u_PCB -> MX_Only:MXOnly-1U-NoLED
- SW60: renamed from SW61; value Enter -> up arrow; footprint Button_Switch_Keyboard:SW_Cherry_MX_1.00u_PCB -> MX_Only:MXOnly-1U-NoLED
- SW63: value Shift -> Ctrl; footprint Button_Switch_Keyboard:SW_Cherry_MX_1.00u_PCB -> MX_Only:MXOnly-1.25U-NoLED
- SW64: value Z -> Win; footprint Button_Switch_Keyboard:SW_Cherry_MX_1.00u_PCB -> MX_Only:MXOnly-1.25U-NoLED
- SW65: value X -> Alt; footprint Button_Switch_Keyboard:SW_Cherry_MX_1.00u_PCB -> MX_Only:MXOnly-1.25U-NoLED
- SW66: renamed from SW68; value B -> Space bar; footprint Button_Switch_Keyboard:SW_Cherry_MX_1.00u_PCB -> MX_Only:MXOnly-6.25U-NoLED
- SW67: renamed from SW71; value , -> Alt; footprint Button_Switch_Keyboard:SW_Cherry_MX_1.00u_PCB -> MX_Only:MXOnly-1U-NoLED
- SW68: renamed from SW72; value . -> Fn; footprint Button_Switch_Keyboard:SW_Cherry_MX_1.00u_PCB -> MX_Only:MXOnly-1U-NoLED
- SW69: renamed from SW73; value / -> right Ctrl; footprint Button_Switch_Keyboard:SW_Cherry_MX_1.00u_PCB -> MX_Only:MXOnly-1U-NoLED
- SW7: value F4 -> $ 4; footprint Button_Switch_Keyboard:SW_Cherry_MX_1.00u_PCB -> MX_Only:MXOnly-1U-NoLED
- SW70: value M -> left arrow; footprint Button_Switch_Keyboard:SW_Cherry_MX_1.00u_PCB -> MX_Only:MXOnly-1U-NoLED
- SW71: renamed from SW74; value r Shift -> down arrow; footprint Button_Switch_Keyboard:SW_Cherry_MX_1.00u_PCB -> MX_Only:MXOnly-1U-NoLED
- SW72: renamed from SW75; value Up Arrow -> right arrow; footprint Button_Switch_Keyboard:SW_Cherry_MX_1.00u_PCB -> MX_Only:MXOnly-1U-NoLED
- SW73: renamed from SW76; footprint Button_Switch_Keyboard:SW_Cherry_MX_1.00u_PCB -> MX_Only:MXOnly-1U-NoLED
- SW8: value F5 -> % 5; footprint Button_Switch_Keyboard:SW_Cherry_MX_1.00u_PCB -> MX_Only:MXOnly-1U-NoLED
- SW9: value F6 -> ^ 6; footprint Button_Switch_Keyboard:SW_Cherry_MX_1.00u_PCB -> MX_Only:MXOnly-1U-NoLED
- moved SW32 284.3 mm to (342.1, 81.0)
- moved SW47 260.4 mm to (342.1, 100.0)
- moved D3 254.5 mm to (34.1, 65.9), turned to 90 degrees
- moved SW16 247.3 mm to (294.5, 61.9)
- moved D17 242.1 mm to (38.9, 84.9), turned to 90 degrees
- moved SW30 239.5 mm to (299.2, 81.0)
- moved SW62 239.3 mm to (342.1, 119.1)
- moved D4 236.9 mm to (53.2, 65.9), turned to 90 degrees
- moved D33 232.3 mm to (41.3, 104.0), turned to 90 degrees
- moved SW13 226.8 mm to (227.8, 61.9)
- moved SW45 223.3 mm to (292.1, 100.0)
- moved D63 222.6 mm to (36.5, 142.1), turned to 90 degrees
- moved SW73 220.5 mm to (342.1, 138.1)
- moved D48 220.4 mm to (46.0, 123.0), turned to 90 degrees
- moved D18 219.8 mm to (62.7, 84.9), turned to 90 degrees
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- renumbered C3 to C1, C4 to C2, C5 to C3, C6 to C4, C7 to C5, C1 to C6, C2 to C7, D9 to D10, D10 to D11, D11 to D12, D12 to D13, D13 to D14, D14 to D15, D15 to D16, D18 to D17, D19 to D18, D20 to D19, D21 to D20, D22 to D21, D23 to D22, D24 to D23, D25 to D24, D26 to D25, D27 to D26, D28 to D27, D29 to D28, D30 to D29, D2 to D3, D31 to D30, D3 to D4, D4 to D5, D5 to D6, D61 to D62, D62 to D63, D63 to D64, D70 to D67, D6 to D7, D73 to D71, D74 to D72, D75 to D73, D7 to D8, D8 to D9, R3 to R4, R4 to R5, R5 to R6, U3 to U2, U2 to U3
Connections:
- D6 pad 1: ROT_ENC_ROW -> Net-(D6-K)
- D6 pad 2: Net-(D5-A) (its old number) -> ROT_ENC_ROW
- SW2 pad A: Net-(R7-Pad1) -> ROT_ENC_A
- SW2 pad B: Net-(R6-Pad1) -> ROT_ENC_B
- SW6 pad 1: Net-(D5-A) (its old number) -> Net-(D6-K)
- SW65 pad 1: Net-(D64-A) (its old number) -> Net-(D65-A)
- SW66 pad 1: Net-(D67-A) (its old number) -> Net-(D66-A)
- SW68 pad 1: Net-(D71-A) (its old number) -> Net-(D68-A)
- SW69 pad 1: Net-(D72-A) (its old number) -> Net-(D69-A)
- SW70 pad 1: Net-(D69-A) -> Net-(D70-A)
- SW70 pad 2: col7 -> col11
- U2 pad 4: unconnected-(U3-PC15-Pad4) -> Net-(D2-A)

Commit message: routed matrix
Parts:
- removed the D46 at (319.9, 104.0)
- removed the D65 at (84.1, 142.1)
- removed the D68 at (243.7, 142.0)
- added D17: D, Diode_SMD:D_SOD-123, B.Cu at (331.0, 67.5)
- added D47: D, Diode_SMD:D_SOD-123, B.Cu at (319.9, 104.0)
- added D67: D, Diode_SMD:D_SOD-123, B.Cu at (155.6, 142.1)
- added D70: D, Diode_SMD:D_SOD-123, B.Cu at (262.7, 142.1)
- moved D66 71.4 mm to (84.1, 142.1)
- moved U2 48.7 mm to (141.3, 135.7)
- moved D69 19.0 mm to (243.7, 142.1)
- moved SW2 12.3 mm to (338.8, 53.1), turned to -90 degrees
- turned D6 to -90 degrees
- renumbered D17 to D18, D18 to D19, D19 to D20, D20 to D21, D21 to D22, D22 to D23, D23 to D24, D24 to D25, D25 to D26, D26 to D27, D27 to D28, D28 to D29, D29 to D30, D30 to D31, D31 to D32, D32 to D33, D33 to D34, D34 to D35, D35 to D36, D36 to D37, D37 to D38, D38 to D39, D39 to D40, D40 to D41, D41 to D42, D42 to D43, D43 to D44, D44 to D45, D45 to D46, D47 to D48, D48 to D49, D49 to D50, D50 to D51, D51 to D52, D52 to D53, D53 to D54, D54 to D55, D55 to D56, D56 to D57, D57 to D58, D58 to D59, D59 to D60, D60 to D61, D61 to D62, D62 to D63, D63 to D64, D64 to D65, D67 to D68, D70 to D71, D71 to D72, D72 to D73, D73 to D74
Connections:
- D10 pad 1: ROT_ENC_ROW -> row0
- D11 pad 1: ROT_ENC_ROW -> row0
- D12 pad 1: ROT_ENC_ROW -> row0
- D13 pad 1: ROT_ENC_ROW -> row0
- D14 pad 1: ROT_ENC_ROW -> row0
- D15 pad 1: ROT_ENC_ROW -> row0
- D16 pad 1: ROT_ENC_ROW -> row0
- D3 pad 1: ROT_ENC_ROW -> row0
- D4 pad 1: ROT_ENC_ROW -> row0
- D5 pad 1: ROT_ENC_ROW -> row0
- D6 pad 2: ROT_ENC_ROW -> row0
- D7 pad 1: ROT_ENC_ROW -> row0
- D8 pad 1: ROT_ENC_ROW -> row0
- D9 pad 1: ROT_ENC_ROW -> row0
- SW65 pad 1: Net-(D65-A) (its old number) -> Net-(D66-A)
- SW66 pad 1: Net-(D66-A) -> Net-(D67-A)
- SW68 pad 1: Net-(D68-A) (its old number) -> Net-(D69-A)
- SW69 pad 1: Net-(D69-A) -> Net-(D70-A)
Routing:
- net row4: track 0.00 -> 302.4 mm
- net row1: track 0.00 -> 300.0 mm
- net row2: track 0.00 -> 297.7 mm
- net row0: track 0.00 -> 295.2 mm
- net row3: track 0.00 -> 292.9 mm
- net col1: track 0.00 -> 95.0 mm
- net col10: track 0.00 -> 94.1 mm
- net col9: track 0.00 -> 93.7 mm
- net col2: track 0.00 -> 92.2 mm
- net col8: track 0.00 -> 92.0 mm
- net col11: track 0.00 -> 92.0 mm
- net col12: track 0.00 -> 92.0 mm
- net col5: track 0.00 -> 87.0 mm
- net col0: track 0.00 -> 85.1 mm
- net col6: track 0.00 -> 67.0 mm
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
Commit message: updated
Parts:
- removed the R6 at (161.2, 179.3)
- removed the R7 at (161.2, 182.2)
- removed the R7 at (178.0, 178.9)
- added R7: 5.1k, Resistor_SMD:R_0805_2012Metric_Pad1.20x1.40mm_HandSolder, F.Cu at (61.1, 96.8)
- D2: moved to F.Cu
- F1: footprint Fuse:Fuse_0805_2012Metric_Pad1.15x1.40mm_HandSolder -> Inductor_SMD:L_0603_1608Metric
- FB1: footprint Ferrite_THT:LairdTech_28C0236-0JW-10 -> Inductor_SMD:L_0603_1608Metric; moved to F.Cu
- moved R6 157.9 mm to (50.0, 64.3), turned to -90 degrees
- moved R4 157.3 mm to (44.5, 65.1), turned to -90 degrees
- moved D2 155.6 mm to (31.8, 100.8)
- moved F1 154.0 mm to (44.5, 61.1), turned to -90 degrees
- moved U1 146.5 mm to (53.2, 73.0)
- moved U3 145.7 mm to (47.4, 64.2), turned to 0 degrees
- moved R1 135.2 mm to (59.5, 75.4), turned to -90 degrees
- moved D1 132.6 mm to (61.9, 73.4), turned to 90 degrees
- moved C6 131.5 mm to (44.5, 69.1), turned to -90 degrees
- moved C7 121.7 mm to (59.5, 71.4), turned to 90 degrees
- moved SW1 83.0 mm to (214.3, 137.3), turned to 0 degrees
- moved C13 80.6 mm to (203.2, 138.1), turned to 0 degrees
- moved C12 78.7 mm to (203.2, 140.5), turned to 0 degrees
- moved Y1 78.0 mm to (198.1, 139.0)
- moved C1 74.2 mm to (202.4, 131.0), turned to -90 degrees
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Connections:
- net Net-(D2-A) renamed PC15
- net Net-(U2-PF0) renamed XTAL_IN
- net Net-(U2-PF1) renamed XTAL_OUT
- R4 pad 1: D+ -> /USB CC1
- USB1 pad 4: D+ -> /USB CC1
Routing:
- net row4: track 302.4 -> 0.09 mm
- net GND: track 0.00 -> 270.9 mm, vias 0 -> 9
- net +3.3V: track 0.00 -> 252.2 mm, vias 0 -> 2
- net D-: track 0.00 -> 192.6 mm
- net D+: track 0.00 -> 191.9 mm
- net PC15: track 0.00 -> 183.3 mm, vias 0 -> 3
- net row0: track 295.2 -> 333.4 mm, vias 0 -> 2
- net BOOT0: track 0.00 -> 36.6 mm, vias 0 -> 2
- net Net-(D2-K): track 0.00 -> 35.8 mm, vias 0 -> 2
- net VBUS: track 0.00 -> 27.2 mm, vias 0 -> 2
- net Net-(F1-Pad1): track 0.00 -> 10.6 mm
- net /USB CC1: track 0.00 -> 6.63 mm
- net Net-(D69-A): track 0.00 -> 5.12 mm
- net Net-(D1-K): track 0.00 -> 2.62 mm
- net row2: track 297.7 -> 297.9 mm, vias 0 -> 4
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